Commit message: bug fixed

File: rl_project_dejulio/urdf/kuka_iiwa/kuka_iiwa_macro_ctrl.xacro (robot description, xacro)
@@ -40,5 +40,5 @@
         <origin xyz="0 0 0" rpy="0 0 0"/>
         <geometry>
-          <mesh filename="package://kuka_iiwa_support/meshes/iiwa7/visual/link_0.stl"/>
+          <mesh filename="package://rl_project_dejulio/meshes/kuka_iiwa/iiwa7/visual/link_0.stl"/>
         </geometry>
         <material name="Grey"/>
@@ -47,5 +47,5 @@
         <origin xyz="0 0 0" rpy="0 0 0"/>
         <geometry>
-          <mesh filename="package://kuka_iiwa_support/meshes/iiwa7/collision/link_0.stl"/>
+          <mesh filename="package://rl_project_dejulio/meshes/kuka_iiwa/iiwa7/collision/link_0.stl"/>
         </geometry>
         <material name="Grey"/>
@@ -139,5 +139,5 @@
         <origin xyz="0 0 -0.026" rpy="0 0 0"/>
         <geometry>
-          <mesh filename="package://kuka_iiwa_support/meshes/iiwa7/visual/link_3.stl"/>
+          <mesh filename="package://rl_project_dejulio/meshes/kuka_iiwa/iiwa7/visual/link_3.stl"/>
         </geometry>
         <material name="Orange"/>
@@ -146,5 +146,5 @@
         <origin xyz="0 0 -0.026" rpy="0 0 0"/>
         <geometry>
-          <mesh filename="package://kuka_iiwa_support/meshes/iiwa7/collision/link_3.stl"/>
+          <mesh filename="package://rl_project_dejulio/meshes/kuka_iiwa/iiwa7/collision/link_3.stl"/>
         </geometry>
         <material name="Orange"/>
